File: kicad/SMD2WII.kicad_pcb (KiCad board)
At the start: 2 copper layers, 31.1 x 44.5 mm, 13 parts, among them J2 DB9_Male, J3 Conn_01x06_Pin, U1 ATmega8A-A

Commit message: PCB confirmed working. Improved position of decoupling capacitor on PCB. Resistor value for green LED changed from 400 Ohm to 4.7k (YMMV).
Parts:
- moved C2 2.17 mm to (106.8, 83.7), turned to -90 degrees
Routing:
- net VCC: track 111.7 -> 108.5 mm
- net GND: track 43.0 -> 44.0 mm, vias 2 -> 1
Changed lines of the file:
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@@
     (property "ki_keywords" "R res resistor")
     (attr smd)
-    (fp_text reference "R3" (at 0 -1.82 90) (layer "F.SilkS")
+    (fp_text reference "R3" (at 0 1.8 90) (layer "F.SilkS")
         (effects (font (size 1 1) (thickness 0.15)))
     )
@@
   )
   (footprint "Capacitor_SMD:C_1206_3216Metric_Pad1.33x1.80mm_HandSolder" (layer "F.Cu")
-    (at 105.3 85.3)
+    (at 106.8 83.7375 -90)
     (descr "Capacitor SMD 1206 (3216 Metric), square (rectangular) end terminal, IPC_7351 nominal with elongated pad for handsoldering. (Body size source: IPC-SM-782 page 76, https://www.pcb-3d.com/wordpress/wp-content/uploads/ipc-sm-782a_amendment_1_and_2.pdf), generated with kicad-footprint-generator")
     (tags "capacitor handsolder")
@@
     (property "ki_keywords" "cap capacitor")
     (attr smd)
-    (fp_text reference "C2" (at 0 -1.85) (layer "F.SilkS")
-        (effects (font (size 1 1) (thickness 0.15)))
-    )
-    (fp_text value "0.1uF" (at 0 1.85) (layer "F.Fab")
-        (effects (font (size 1 1) (thickness 0.15)))
-    )
-    (fp_text user "${REFERENCE}" (at 0 0) (layer "F.Fab")
+    (fp_text reference "C2" (at 0 -1.85 90) (layer "F.SilkS")
+        (effects (font (size 1 1) (thickness 0.15)))
+    )
+    (fp_text value "0.1uF" (at 0 1.85 90) (layer "F.Fab")
+        (effects (font (size 1 1) (thickness 0.15)))
+    )
+    (fp_text user "${REFERENCE}" (at 0 0 90) (layer "F.Fab")
         (effects (font (size 0.8 0.8) (thickness 0.12)))
     )
@@
     (fp_line (start 1.6 0.8) (end -1.6 0.8)
       (stroke (width 0.1) (type solid)) (layer "F.Fab"))
-    (pad "1" smd roundrect (at -1.5625 0) (size 1.325 1.8) (layers "F.Cu" "F.Paste" "F.Mask") (roundrect_rratio 0.1886792453)
+    (pad "1" smd roundrect (at -1.5625 0 270) (size 1.325 1.8) (layers "F.Cu" "F.Paste" "F.Mask") (roundrect_rratio 0.1886792453)
       (net 1 "VCC") (pintype "passive"))
-    (pad "2" smd roundrect (at 1.5625 0) (size 1.325 1.8) (layers "F.Cu" "F.Paste" "F.Mask") (roundrect_rratio 0.1886792453)
+    (pad "2" smd roundrect (at 1.5625 0 270) (size 1.325 1.8) (layers "F.Cu" "F.Paste" "F.Mask") (roundrect_rratio 0.1886792453)
       (net 2 "GND") (pintype "passive"))
     (model "${KICAD6_3DMODEL_DIR}/Capacitor_SMD.3dshapes/C_1206_3216Metric.wrl"
@@
   (segment (start 124.8 85.35) (end 124.8 83) (width 0.5) (layer "F.Cu") (net 1))
   (segment (start 110.63 82.17) (end 103.7 82.17) (width 1) (layer "F.Cu") (net 1))
-  (segment (start 103.7375 82.2075) (end 103.7 82.17) (width 0.35) (layer "F.Cu") (net 1))
-  (segment (start 103.7375 85.3) (end 103.7375 82.2075) (width 0.5) (layer "F.Cu") (net 1))
   (segment (start 113.9 72.7) (end 113.45 73.15) (width 0.5) (layer "F.Cu") (net 1))
   (segment (start 110.63 82.17) (end 111.5 81.3) (width 0.5) (layer "F.Cu") (net 1))
@@
   (segment (start 109.2 93.81066) (end 109.2 91.1) (width 1) (layer "F.Cu") (net 2))
   (segment (start 113.45 69.05) (end 113.1 69.4) (width 0.5) (layer "F.Cu") (net 2))
-  (segment (start 106.8625 85.3) (end 109.2 85.3) (width 0.5) (layer "F.Cu") (net 2))
   (segment (start 109.2 91.1) (end 109.2 87.2) (width 1) (layer "F.Cu") (net 2))
   (segment (start 111.3 85.4125) (end 109.3125 85.4125) (width 0.5) (layer "F.Cu") (net 2))
@@
   (segment (start 111.5 83.6) (end 109.9 83.6) (width 0.5) (layer "F.Cu") (net 2))
   (segment (start 114.7 71.2) (end 114.7 74.6) (width 0.5) (layer "F.Cu") (net 2))
+  (segment (start 106.8 85.3) (end 109.2 85.3) (width 0.5) (layer "F.Cu") (net 2))
   (segment (start 113.9 75.4) (end 113.9 79.7) (width 0.5) (layer "F.Cu") (net 2))
   (segment (start 114.35 69.05) (end 114.7 69.4) (width 0.5) (layer "F.Cu") (net 2))
   (segment (start 109.3125 85.4125) (end 109.2 85.3) (width 0.35) (layer "F.Cu") (net 2))
+  (segment (start 114.35 69.05) (end 113.45 69.05) (width 0.5) (layer "F.Cu") (net 2))
   (segment (start 109.9 83.6) (end 109.7 83.8) (width 0.5) (layer "F.Cu") (net 2))
   (segment (start 116.9 85.4125) (end 116.9 83.2) (width 0.35) (layer "F.Cu") (net 2))
@@
   (segment (start 113.9 81.2) (end 111.5 83.6) (width 0.5) (layer "F.Cu") (net 2))
   (segment (start 113.1 69.4) (end 113.1 71.2) (width 0.5) (layer "F.Cu") (net 2))
-  (via (at 113.85 69.05) (size 1) (drill 0.5) (layers "F.Cu" "B.Cu") (net 2))
   (via (at 116.9 83.2) (size 0.8) (drill 0.4) (layers "F.Cu" "B.Cu") (net 2))
   (segment (start 121.65 91.2495) (end 121.5995 91.3) (width 0.5) (layer "F.Cu") (net 3))
