File: kicad/SMD2WII.kicad_sch (KiCad schematic)
At the start: 13 parts, among them J2 DB9_Male, J3 Conn_01x06_Pin, U1 ATmega8A-A

Commit message: Swap MISO <=> MOSI.
Connections:
- net MISO: now also J3.4 (Pin_4), U1.16 (PB4); no longer J3.3 (Pin_3), U1.15 (PB3)
- net MOSI: now also J3.3 (Pin_3), U1.15 (PB3); no longer J3.4 (Pin_4), U1.16 (PB4)
Changed lines of the file:
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@@
     (effects (font (size 1.27 1.27)) (justify left bottom))
   )
-  (label "MISO" (at 147.32 74.93 0) (fields_autoplaced)
+  (label "MOSI" (at 147.32 74.93 0) (fields_autoplaced)
     (effects (font (size 1.27 1.27)) (justify left bottom))
   )
@@
     (effects (font (size 1.27 1.27)) (justify left bottom))
   )
-  (label "MOSI" (at 157.48 52.07 0) (fields_autoplaced)
+  (label "MISO" (at 157.48 52.07 0) (fields_autoplaced)
     (effects (font (size 1.27 1.27)) (justify left bottom))
   )
@@
     (effects (font (size 1.27 1.27)) (justify left bottom))
   )
-  (label "MOSI" (at 147.32 77.47 0) (fields_autoplaced)
+  (label "MISO" (at 147.32 77.47 0) (fields_autoplaced)
     (effects (font (size 1.27 1.27)) (justify left bottom))
   )
@@
     (effects (font (size 1.27 1.27)) (justify left bottom))
   )
-  (label "MISO" (at 157.48 54.61 0) (fields_autoplaced)
+  (label "MOSI" (at 157.48 54.61 0) (fields_autoplaced)
     (effects (font (size 1.27 1.27)) (justify left bottom))
   )

Commit message: Connect RESET to VCC instead of GND.
Connections:
- net GND: no longer R3.1
- net VCC: now also R3.1
Changed lines of the file:
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@@
-    )
-  )
-  (symbol (lib_name "GND_3") (lib_id "power:GND") (at 105.41 49.53 180) (unit 1)
-    (in_bom yes) (on_board yes) (dnp no) (fields_autoplaced)
-    (property "Reference" "#PWR0113" (at 105.41 43.18 0)
-      (effects (font (size 1.27 1.27)) hide)
-    )
-    (property "Value" "GND" (at 105.41 44.45 0)
-      (effects (font (size 1.27 1.27)))
-    )
-    (property "Footprint" "" (at 105.41 49.53 0)
-      (effects (font (size 1.27 1.27)) hide)
-    )
-    (property "Datasheet" "" (at 105.41 49.53 0)
-      (effects (font (size 1.27 1.27)) hide)
-    )
-    (pin "1")
-    (instances
-      (project "SMD2WII"
-        (path "/7c85da91-93f1-4d04-8833-88ec1b827959"
-          (reference "#PWR0113") (unit 1)
-        )
-      )
     )
   )
@@
         )
       )
+    )
+  )
+  (symbol (lib_id "power:VCC") (at 105.41 49.53 0) (unit 1)
+    (in_bom yes) (on_board yes) (dnp no) (fields_autoplaced)
+    (property "Reference" "#PWR04" (at 105.41 53.34 0)
+      (effects (font (size 1.27 1.27)) hide)
+    )
+    (property "Value" "VCC" (at 105.41 44.45 0)
+      (effects (font (size 1.27 1.27)))
+    )
+    (property "Footprint" "" (at 105.41 49.53 0)
+      (effects (font (size 1.27 1.27)) hide)
+    )
+    (property "Datasheet" "" (at 105.41 49.53 0)
+      (effects (font (size 1.27 1.27)) hide)
+    )
+    (pin "1")
+    (instances
+      (project "SMD2WII"
+        (path "/7c85da91-93f1-4d04-8833-88ec1b827959"
+          (reference "#PWR04") (unit 1)
+        )
+      )

Commit message: PCB confirmed working. Improved position of decoupling capacitor on PCB. Resistor value for green LED changed from 400 Ohm to 4.7k (YMMV).
Parts:
- R4: value 400 -> 390
- R5: value 400 -> 4.7k
Changed lines of the file:
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@@
       (effects (font (size 1.27 1.27)) (justify left))
     )
-    (property "Value" "400" (at 144.78 128.2699 0)
+    (property "Value" "4.7k" (at 144.78 128.2699 0)
       (effects (font (size 1.27 1.27)) (justify left))
     )
@@
       (effects (font (size 1.27 1.27)) (justify left))
     )
-    (property "Value" "400" (at 157.48 128.27 0)
+    (property "Value" "390" (at 157.48 128.27 0)
       (effects (font (size 1.27 1.27)) (justify left))
     )
